Commit message: Update real hardware
Adapts xacro for real hardware

File: urdf/marta.xacro (robot description, xacro)
@@ -7,6 +7,11 @@
 <xacro:include filename="$(find marta_description)/urdf/IMU.xacro" />
 <xacro:include filename="$(find marta_description)/urdf/marta_joints.xacro" />
-<xacro:imu_sensor parent="base_link" ns="marta" origin="-5.76e-3 -53.277e-3 -48.948e-3 0 0 0"/>
-<xacro:camera_sensor parent="head_1" camera_name="front_camera" ns="marta" origin="-0.02060 -0.050864 0.047202 0 0 -1.57"/>
+<!-- Define o parâmetro "use_sim" -->
+<xacro:property name="use_sim" value="true" />
+<!-- Adiciona o imu_sensor e camera_sensor apenas se use_sim for true -->
+<xacro:if value="${use_sim}">
+  <xacro:imu_sensor parent="base_link" ns="marta" origin="-5.76e-3 -53.277e-3 -48.948e-3 0 0 0"/>
+  <xacro:camera_sensor parent="head_1" camera_name="front_camera" ns="marta" origin="-0.02060 -0.050864 0.047202 0 0 -1.57"/>
+</xacro:if>
 <link name="base_link">
   <inertial>
@@ -447,3 +452,15 @@
   </collision>
 </link>
+<link name="imu_position">
+  <inertial>
+    <origin xyz="-5.76e-3 53.277e-3 48.948e-3" rpy="0 0 0" />
+    <mass value="0.0" />
+    <inertia ixx="0.0" iyy="0.0" izz="0.0" ixy="0.0" iyz="0.0" ixz="0.0" />
+  </inertial>
+</link>
+<joint name="imu_joint" type="fixed">
+  <parent link="base_link" />
+  <child link="imu_position" />
+  <origin xyz="-5.76e-3 53.277e-3 48.948e-3" rpy="0 0 0" />
+</joint>
 </robot>

File: urdf/marta_joints.xacro (robot description, xacro)
@@ -112,5 +112,5 @@
   <parent link="base_link"/>
   <child link="l_shoulder_1"/>
-  <axis xyz="0.0 -1.0 0.0"/>
+  <axis xyz="0.0 1.0 0.0"/>
   <!-- <dynamics damping="0.1" /> -->
   <limit lower="-3.14159" upper="3.14159" effort="1000.0" velocity="0.01"/>
@@ -120,5 +120,5 @@
   <parent link="base_link"/>
   <child link="r_shoulder_1"/>
-  <axis xyz="-0.0 -1.0 -0.0"/>
+  <axis xyz="-0.0 1.0 -0.0"/>
   <!-- <dynamics damping="0.1" /> -->
   <limit lower="-3.14159" upper="3.14159" effort="1000.0" velocity="0.01"/>
@@ -152,5 +152,5 @@
   <parent link="r_arm_1"/>
   <child link="r_hand_1"/>
-  <axis xyz="0.0 -1.0 -0.0"/>
+  <axis xyz="0.0 1.0 -0.0"/>
   <!-- <dynamics damping="0.1" /> -->
   <limit lower="-3.14159" upper="3.14159" effort="1000.0" velocity="0.01"/>
@@ -160,5 +160,5 @@
   <parent link="l_arm_1"/>
   <child link="l_hand_1"/>
-  <axis xyz="-0.0 -1.0 0.0"/>
+  <axis xyz="-0.0 1.0 0.0"/>
   <!-- <dynamics damping="0.1" /> -->
   <limit lower="-3.14159" upper="3.14159" effort="1000.0" velocity="0.01"/>
