Commit message: Modelo de servo MX-28 e escala de massa do tronco
- controller_mx28.yaml (p = 12,74 N.m/rad, tese do Maximo)
- args torso_mass_scale, implicit_damping e joint_velocity (o limite de
  0,01 rad/s do URDF freava as juntas)

File: urdf/marta.xacro (robot description, xacro)
@@ -46,4 +46,16 @@
 <xacro:arg name="imu_gyro_bias"   default="0.0"/>
 <xacro:arg name="foot_collision"  default="box"/>
+<!-- Escala da massa do tronco (base_link); a inercia escala junto (mesma forma,
+     densidade proporcional). 1.0 = modelo original. Experimento de massa. -->
+<xacro:arg name="torso_mass_scale" default="1.0"/>
+<!-- Integra o amortecimento de junta (joint_damping) de forma IMPLICITA no ODE
+     (implicitSpringDamper). O explicito foi instavel (README, achado D). Usado
+     pelo modelo de servo MX-28 (plano_comparacao_darwin.md §3). -->
+<xacro:arg name="implicit_damping" default="false"/>
+<!-- Limite de velocidade das juntas [rad/s]. O original e 0,01; o Gazebo zera o
+     esforco que empurra a junta no sentido do movimento acima dele (so deixa
+     frear). MX-28 a 12 V: 5,76 rad/s em vazio. -->
+<xacro:arg name="joint_velocity" default="0.01"/>
+<xacro:property name="joint_velocity" value="$(arg joint_velocity)"/>
 <xacro:property name="foot_mu"         value="$(arg foot_mu)"/>
 <xacro:property name="body_mu1"        value="$(arg body_mu1)"/>
@@ -54,6 +66,29 @@
 <xacro:property name="joint_damping"   value="$(arg joint_damping)"/>
 <xacro:property name="joint_friction"  value="$(arg joint_friction)"/>
+<xacro:property name="torso_mass_scale" value="$(arg torso_mass_scale)"/>
 <xacro:include filename="$(find marta_description)/urdf/materials.xacro" />
 <xacro:include filename="$(find marta_description)/urdf/marta.trans" />
+<xacro:if value="$(arg implicit_damping)">
+  <gazebo reference="head_pan_link"><implicitSpringDamper>true</implicitSpringDamper></gazebo>
+  <gazebo reference="head_tilt_link"><implicitSpringDamper>true</implicitSpringDamper></gazebo>
+  <gazebo reference="r_hip_yaw_link"><implicitSpringDamper>true</implicitSpringDamper></gazebo>
+  <gazebo reference="l_hip_yaw_link"><implicitSpringDamper>true</implicitSpringDamper></gazebo>
+  <gazebo reference="l_hip_roll_link"><implicitSpringDamper>true</implicitSpringDamper></gazebo>
+  <gazebo reference="r_hip_roll_link"><implicitSpringDamper>true</implicitSpringDamper></gazebo>
+  <gazebo reference="r_hip_pitch_link"><implicitSpringDamper>true</implicitSpringDamper></gazebo>
+  <gazebo reference="l_hip_pitch_link"><implicitSpringDamper>true</implicitSpringDamper></gazebo>
+  <gazebo reference="r_knee_link"><implicitSpringDamper>true</implicitSpringDamper></gazebo>
+  <gazebo reference="l_knee_link"><implicitSpringDamper>true</implicitSpringDamper></gazebo>
+  <gazebo reference="l_ank_pitch_link"><implicitSpringDamper>true</implicitSpringDamper></gazebo>
+  <gazebo reference="r_ank_pitch_link"><implicitSpringDamper>true</implicitSpringDamper></gazebo>
+  <gazebo reference="r_ank_roll_link"><implicitSpringDamper>true</implicitSpringDamper></gazebo>
+  <gazebo reference="l_sho_pitch_link"><implicitSpringDamper>true</implicitSpringDamper></gazebo>
+  <gazebo reference="r_sho_pitch_link"><implicitSpringDamper>true</implicitSpringDamper></gazebo>
+  <gazebo reference="l_sho_roll_link"><implicitSpringDamper>true</implicitSpringDamper></gazebo>
+  <gazebo reference="r_sho_roll_link"><implicitSpringDamper>true</implicitSpringDamper></gazebo>
+  <gazebo reference="l_ank_roll_link"><implicitSpringDamper>true</implicitSpringDamper></gazebo>
+  <gazebo reference="r_el_link"><implicitSpringDamper>true</implicitSpringDamper></gazebo>
+  <gazebo reference="l_el_link"><implicitSpringDamper>true</implicitSpringDamper></gazebo>
+</xacro:if>
 <xacro:include filename="$(find marta_description)/urdf/marta.gazebo" />
 <xacro:include filename="$(find marta_description)/urdf/camera.xacro" />
@@ -74,6 +109,6 @@
   <inertial>
     <origin xyz="5.4347537332971534e-05 -0.0007644260033313482 -0.006523313454687187" rpy="0 0 0"/>
-    <mass value="2.9663080742707644"/>
-    <inertia ixx="0.011903" iyy="0.0138" izz="0.007909" ixy="-0.000103" iyz="-5e-06" ixz="-0.000518"/>
+    <mass value="${2.9663080742707644 * torso_mass_scale}"/>
+    <inertia ixx="${0.011903 * torso_mass_scale}" iyy="${0.0138 * torso_mass_scale}" izz="${0.007909 * torso_mass_scale}" ixy="${-0.000103 * torso_mass_scale}" iyz="${-5e-06 * torso_mass_scale}" ixz="${-0.000518 * torso_mass_scale}"/>
   </inertial>
   <visual>

File: urdf/marta_joints.xacro (robot description, xacro)
@@ -10,5 +10,5 @@
   <axis xyz="-0.0 0.0 -1.0"/>
   <dynamics damping="${joint_damping}" friction="${joint_friction}"/>
-  <limit lower="-3.14159" upper="3.14159" effort="${joint_effort}" velocity="0.01"/>
+  <limit lower="-3.14159" upper="3.14159" effort="${joint_effort}" velocity="${joint_velocity}"/>
 </joint>
 <joint name="head_tilt_link" type="revolute">
@@ -18,5 +18,5 @@
   <axis xyz="-0.0 -1.0 -0.0"/>
   <dynamics damping="${joint_damping}" friction="${joint_friction}"/>
-  <limit lower="-3.14159" upper="3.14159" effort="${joint_effort}" velocity="0.01"/>
+  <limit lower="-3.14159" upper="3.14159" effort="${joint_effort}" velocity="${joint_velocity}"/>
 </joint>
 <joint name="r_hip_yaw_link" type="revolute">
@@ -26,5 +26,5 @@
   <axis xyz="-0.0 0.0 -1.0"/>
   <dynamics damping="${joint_damping}" friction="${joint_friction}"/>
-  <limit lower="-3.14159" upper="3.14159" effort="${joint_effort}" velocity="0.01"/>
+  <limit lower="-3.14159" upper="3.14159" effort="${joint_effort}" velocity="${joint_velocity}"/>
 </joint>
 <joint name="l_hip_yaw_link" type="revolute">
@@ -34,5 +34,5 @@
   <axis xyz="0.0 0.0 -1.0"/>
   <dynamics damping="${joint_damping}" friction="${joint_friction}"/>
-  <limit lower="-3.14159" upper="3.14159" effort="${joint_effort}" velocity="0.01"/>
+  <limit lower="-3.14159" upper="3.14159" effort="${joint_effort}" velocity="${joint_velocity}"/>
 </joint>
 <joint name="l_hip_roll_link" type="revolute">
@@ -42,5 +42,5 @@
   <axis xyz="1.0 -0.0 0.0"/>
   <dynamics damping="${joint_damping}" friction="${joint_friction}"/>
-  <limit lower="-3.14159" upper="3.14159" effort="${joint_effort}" velocity="0.01"/>
+  <limit lower="-3.14159" upper="3.14159" effort="${joint_effort}" velocity="${joint_velocity}"/>
 </joint>
 <joint name="r_hip_roll_link" type="revolute">
@@ -50,5 +50,5 @@
   <axis xyz="1.0 0.0 -0.0"/>
   <dynamics damping="${joint_damping}" friction="${joint_friction}"/>
-  <limit lower="-3.14159" upper="3.14159" effort="${joint_effort}" velocity="0.01"/>
+  <limit lower="-3.14159" upper="3.14159" effort="${joint_effort}" velocity="${joint_velocity}"/>
 </joint>
 <joint name="r_hip_pitch_link" type="revolute">
@@ -58,5 +58,5 @@
   <axis xyz="0.0 1.0 -0.0"/>
   <dynamics damping="${joint_damping}" friction="${joint_friction}"/>
-  <limit lower="-3.14159" upper="3.14159" effort="${joint_effort}" velocity="0.01"/>
+  <limit lower="-3.14159" upper="3.14159" effort="${joint_effort}" velocity="${joint_velocity}"/>
 </joint>
 <joint name="l_hip_pitch_link" type="revolute">
@@ -66,5 +66,5 @@
   <axis xyz="0.0 1.0 0.0"/>
   <dynamics damping="${joint_damping}" friction="${joint_friction}"/>
-  <limit lower="-3.14159" upper="3.14159" effort="${joint_effort}" velocity="0.01"/>
+  <limit lower="-3.14159" upper="3.14159" effort="${joint_effort}" velocity="${joint_velocity}"/>
 </joint>
 <joint name="r_knee_link" type="revolute">
@@ -74,5 +74,5 @@
   <axis xyz="-0.0 1.0 -0.0"/>
   <dynamics damping="${joint_damping}" friction="${joint_friction}"/>
-  <limit lower="-3.14159" upper="3.14159" effort="${joint_effort}" velocity="0.01"/>
+  <limit lower="-3.14159" upper="3.14159" effort="${joint_effort}" velocity="${joint_velocity}"/>
 </joint>
 <joint name="l_knee_link" type="revolute">
@@ -82,5 +82,5 @@
   <axis xyz="0.0 1.0 0.0"/>
   <dynamics damping="${joint_damping}" friction="${joint_friction}"/>
-  <limit lower="-3.14159" upper="3.14159" effort="${joint_effort}" velocity="0.01"/>
+  <limit lower="-3.14159" upper="3.14159" effort="${joint_effort}" velocity="${joint_velocity}"/>
 </joint>
 <joint name="l_ank_pitch_link" type="revolute">
@@ -90,5 +90,5 @@
   <axis xyz="-0.0 1.0 -0.0"/>
   <dynamics damping="${joint_damping}" friction="${joint_friction}"/>
-  <limit lower="-3.14159" upper="3.14159" effort="${joint_effort}" velocity="0.01"/>
+  <limit lower="-3.14159" upper="3.14159" effort="${joint_effort}" velocity="${joint_velocity}"/>
 </joint>
 <joint name="r_ank_pitch_link" type="revolute">
@@ -98,5 +98,5 @@
   <axis xyz="-0.0 1.0 0.0"/>
   <dynamics damping="${joint_damping}" friction="${joint_friction}"/>
-  <limit lower="-3.14159" upper="3.14159" effort="${joint_effort}" velocity="0.01"/>
+  <limit lower="-3.14159" upper="3.14159" effort="${joint_effort}" velocity="${joint_velocity}"/>
 </joint>
 <joint name="r_ank_roll_link" type="revolute">
@@ -106,5 +106,5 @@
   <axis xyz="1.0 0.0 -0.0"/>
   <dynamics damping="${joint_damping}" friction="${joint_friction}"/>
-  <limit lower="-3.14159" upper="3.14159" effort="${joint_effort}" velocity="0.01"/>
+  <limit lower="-3.14159" upper="3.14159" effort="${joint_effort}" velocity="${joint_velocity}"/>
 </joint>
 <joint name="l_sho_pitch_link" type="revolute">
@@ -114,5 +114,5 @@
   <axis xyz="0.0 1.0 0.0"/>
   <dynamics damping="${joint_damping}" friction="${joint_friction}"/>
-  <limit lower="-3.14159" upper="3.14159" effort="${joint_effort}" velocity="0.01"/>
+  <limit lower="-3.14159" upper="3.14159" effort="${joint_effort}" velocity="${joint_velocity}"/>
 </joint>
 <joint name="r_sho_pitch_link" type="revolute">
@@ -122,5 +122,5 @@
   <axis xyz="-0.0 1.0 -0.0"/>
   <dynamics damping="${joint_damping}" friction="${joint_friction}"/>
-  <limit lower="-3.14159" upper="3.14159" effort="${joint_effort}" velocity="0.01"/>
+  <limit lower="-3.14159" upper="3.14159" effort="${joint_effort}" velocity="${joint_velocity}"/>
 </joint>
 <joint name="l_sho_roll_link" type="revolute">
@@ -130,5 +130,5 @@
   <axis xyz="-1.0 -0.0 -0.0"/>
   <dynamics damping="${joint_damping}" friction="${joint_friction}"/>
-  <limit lower="-3.14159" upper="3.14159" effort="${joint_effort}" velocity="0.01"/>
+  <limit lower="-3.14159" upper="3.14159" effort="${joint_effort}" velocity="${joint_velocity}"/>
 </joint>
 <joint name="r_sho_roll_link" type="revolute">
@@ -138,5 +138,5 @@
   <axis xyz="-1.0 0.0 -0.0"/>
   <dynamics damping="${joint_damping}" friction="${joint_friction}"/>
-  <limit lower="-3.14159" upper="3.14159" effort="${joint_effort}" velocity="0.01"/>
+  <limit lower="-3.14159" upper="3.14159" effort="${joint_effort}" velocity="${joint_velocity}"/>
 </joint>
 <joint name="l_ank_roll_link" type="revolute">
@@ -146,5 +146,5 @@
   <axis xyz="1.0 -0.0 0.0"/>
   <dynamics damping="${joint_damping}" friction="${joint_friction}"/>
-  <limit lower="-3.14159" upper="3.14159" effort="${joint_effort}" velocity="0.01"/>
+  <limit lower="-3.14159" upper="3.14159" effort="${joint_effort}" velocity="${joint_velocity}"/>
 </joint>
 <joint name="r_el_link" type="revolute">
@@ -154,5 +154,5 @@
   <axis xyz="0.0 1.0 -0.0"/>
   <dynamics damping="${joint_damping}" friction="${joint_friction}"/>
-  <limit lower="-3.14159" upper="3.14159" effort="${joint_effort}" velocity="0.01"/>
+  <limit lower="-3.14159" upper="3.14159" effort="${joint_effort}" velocity="${joint_velocity}"/>
 </joint>
 <joint name="l_el_link" type="revolute">
@@ -162,5 +162,5 @@
   <axis xyz="-0.0 1.0 0.0"/>
   <dynamics damping="${joint_damping}" friction="${joint_friction}"/>
-  <limit lower="-3.14159" upper="3.14159" effort="${joint_effort}" velocity="0.01"/>
+  <limit lower="-3.14159" upper="3.14159" effort="${joint_effort}" velocity="${joint_velocity}"/>
 </joint>
 </robot>
