Commit message: Knobs de realismo da simulacao e colisao do pe em caixa por padrao
foot_collision (box|mesh): a colisao de malha STL fazia o pe de apoio girar
no ODE e o robo derivar para a esquerda. Inclui knobs de atrito, contato,
torque, damping e ruido de IMU.

File: urdf/IMU.xacro (robot description, xacro)
@@ -1,8 +1,27 @@
 <?xml version="1.0"?>
 <robot xmlns:xacro="http://www.ros.org/wiki/xacro">
-    <xacro:macro name="imu_sensor" params="parent origin ns">
+    <!--
+      gyro_noise  [rad/s]   desvio padrao do ruido gaussiano na velocidade angular
+      accel_noise [m/s^2]   desvio padrao do ruido gaussiano na aceleracao
+      gyro_bias   [rad/s]   bias constante do giroscopio. Atencao: o erro de
+                            regime do filtro complementar e bias * tau, entao com
+                            tau ~ 5 s um bias de 0,01 rad/s vira ~2,9 graus de
+                            offset permanente no pitch estimado.
+      accel_bias  [m/s^2]   bias constante do acelerometro
+      Zero em todos por default, o que reproduz o comportamento anterior. O ruido
+      e aplicado pelo proprio Gazebo no bloco <imu> do SDF, por eixo, o que e
+      mais fiel do que o <gaussianNoise> do plugin (um valor unico para tudo).
+    -->
+    <xacro:macro name="imu_sensor"
+                 params="parent origin ns
+                         gyro_noise:=0.0 accel_noise:=0.0
+                         gyro_bias:=0.0 accel_bias:=0.0">
         <!-- Gazebo sensor configuration -->
         <gazebo reference="${parent}">
             <gravity>true</gravity>
+            <!-- update_rate (taxa de amostragem do sensor) e updateRateHZ (taxa
+                 de publicacao do plugin) precisam ser iguais: com 100 e 10 o
+                 topico saia a 10 Hz, taxa insuficiente para o laco de controle
+                 e para a estimacao de atitude a 100 Hz. -->
             <sensor name="imu_sensor" type="imu">
                 <always_on>true</always_on>
@@ -12,6 +31,11 @@
                 <plugin filename="libgazebo_ros_imu_sensor.so" name="imu_plugin">
                     <topicName>/${ns}/imu</topicName>
-                    <bodyName>imu_link</bodyName>
-                    <updateRateHZ>10.0</updateRateHZ>
+                    <!-- imu_link nao existe no URDF; o sensor esta fixado em
+                         base_link (ver marta.xacro). A pose abaixo rotaciona o
+                         frame de medicao em R_y(pi) em relacao a base_link, o
+                         que e tratado pelo parametro imu_mount_rpy do
+                         torso_attitude_node. -->
+                    <bodyName>base_link</bodyName>
+                    <updateRateHZ>100.0</updateRateHZ>
                     <gaussianNoise>0.0</gaussianNoise>
                     <xyzOffset>0 0 0</xyzOffset>
@@ -20,4 +44,28 @@
                     <initialOrientationAsReference>false</initialOrientationAsReference>
                 </plugin>
+                <imu>
+                    <angular_velocity>
+                        <x><noise type="gaussian">
+                            <mean>${gyro_bias}</mean><stddev>${gyro_noise}</stddev>
+                        </noise></x>
+                        <y><noise type="gaussian">
+                            <mean>${gyro_bias}</mean><stddev>${gyro_noise}</stddev>
+                        </noise></y>
+                        <z><noise type="gaussian">
+                            <mean>${gyro_bias}</mean><stddev>${gyro_noise}</stddev>
+                        </noise></z>
+                    </angular_velocity>
+                    <linear_acceleration>
+                        <x><noise type="gaussian">
+                            <mean>${accel_bias}</mean><stddev>${accel_noise}</stddev>
+                        </noise></x>
+                        <y><noise type="gaussian">
+                            <mean>${accel_bias}</mean><stddev>${accel_noise}</stddev>
+                        </noise></y>
+                        <z><noise type="gaussian">
+                            <mean>${accel_bias}</mean><stddev>${accel_noise}</stddev>
+                        </noise></z>
+                    </linear_acceleration>
+                </imu>
                 <pose>${origin}</pose>
             </sensor>

File: urdf/marta.xacro (robot description, xacro)
@@ -1,4 +1,57 @@
 <?xml version="1.0" ?>
 <robot name="marta" xmlns:xacro="http://www.ros.org/wiki/xacro">
+<!--
+  ============================================================================
+  Knobs de realismo da simulação
+  ============================================================================
+  Todos os defaults reproduzem exatamente o modelo anterior, então nada muda a
+  menos que seja passado na linha de comando do xacro, com UMA exceção:
+  foot_collision, cujo default passou a ser "box" em 2026-10-07 (a colisão de
+  malha fazia o robô girar sozinho para a esquerda; ver docs/README.md, achado
+  I). Campanhas anteriores a essa data rodaram com "mesh". Os knobs servem para
+  degradar a simulação de forma controlada, um fator por vez.
+    foot_mu        1e10   -> atrito do pé. Adimensional; na física real fica
+                            abaixo de ~1,5. Com 1e10 o pé nunca escorrega.
+    body_mu1/2     500/400 -> atrito dos demais links (só importa em colisão)
+    contact_kp/kd  1e6/1e4 -> rigidez e amortecimento do contato do pé
+    joint_effort   1000.0 -> limite de torque das juntas [N·m]. A Marta tem
+                            4,78 kg e precisa de ~2-4 N·m no joelho; um servo
+                            KidSize entrega 2-6 N·m. 1000 é ~200x de margem.
+    joint_damping  0.0    -> atrito viscoso das juntas [N·m·s/rad]
+    joint_friction 0.0    -> atrito de Coulomb das juntas [N·m]
+    imu_gyro_noise 0.0    -> desvio padrão do ruído do giroscópio [rad/s]
+    imu_accel_noise 0.0   -> desvio padrão do ruído do acelerômetro [m/s²]
+    imu_gyro_bias  0.0    -> bias do giroscópio [rad/s]
+    foot_collision box    -> geometria de colisão do pé: "mesh" (STL original)
+                            ou "box" (caixa com a mesma sola: 0,140 x 0,070 m,
+                            fundo em z = -0,037 no frame do link). Com "mesh" o
+                            pé de apoio gira 1-2 graus no chão a cada passo e o
+                            robô deriva ~4 graus/s para a esquerda; com "box",
+                            ~0 e sem lado preferido. O visual segue sendo o STL.
+  NOTA: o terreno é deliberadamente mantido plano e nivelado. O gerador de
+  marcha assume solo plano e altura de CoM constante no LIPM; inclinar ou
+  acidentar o chão violaria a premissa do gerador em vez de testar o
+  estabilizador.
+-->
+<xacro:arg name="foot_mu"         default="1e10"/>
+<xacro:arg name="body_mu1"        default="500"/>
+<xacro:arg name="body_mu2"        default="400"/>
+<xacro:arg name="contact_kp"      default="1000000.0"/>
+<xacro:arg name="contact_kd"      default="10000.0"/>
+<xacro:arg name="joint_effort"    default="1000.0"/>
+<xacro:arg name="joint_damping"   default="0.0"/>
+<xacro:arg name="joint_friction"  default="0.0"/>
+<xacro:arg name="imu_gyro_noise"  default="0.0"/>
+<xacro:arg name="imu_accel_noise" default="0.0"/>
+<xacro:arg name="imu_gyro_bias"   default="0.0"/>
+<xacro:arg name="foot_collision"  default="box"/>
+<xacro:property name="foot_mu"         value="$(arg foot_mu)"/>
+<xacro:property name="body_mu1"        value="$(arg body_mu1)"/>
+<xacro:property name="body_mu2"        value="$(arg body_mu2)"/>
+<xacro:property name="contact_kp"      value="$(arg contact_kp)"/>
+<xacro:property name="contact_kd"      value="$(arg contact_kd)"/>
+<xacro:property name="joint_effort"    value="$(arg joint_effort)"/>
+<xacro:property name="joint_damping"   value="$(arg joint_damping)"/>
+<xacro:property name="joint_friction"  value="$(arg joint_friction)"/>
 <xacro:include filename="$(find marta_description)/urdf/materials.xacro" />
 <xacro:include filename="$(find marta_description)/urdf/marta.trans" />
@@ -11,5 +64,9 @@
 <!-- Adiciona o imu_sensor e camera_sensor apenas se use_sim for true -->
 <xacro:if value="${use_sim}">
-  <xacro:imu_sensor parent="base_link" ns="marta" origin="-5.76e-3 -53.277e-3 -48.948e-3 ${pi} 0 ${pi}"/>
+  <xacro:imu_sensor parent="base_link" ns="marta"
+                    origin="-5.76e-3 -53.277e-3 -48.948e-3 ${pi} 0 ${pi}"
+                    gyro_noise="$(arg imu_gyro_noise)"
+                    accel_noise="$(arg imu_accel_noise)"
+                    gyro_bias="$(arg imu_gyro_bias)"/>
   <xacro:camera_sensor parent="head_1" camera_name="front_camera" ns="marta" origin="0.04060 -0.020864 0.051202 0 0 0"/>
 </xacro:if>
@@ -408,14 +465,25 @@
   </visual>
   <collision>
-    <origin xyz="0.017701 -0.039506 0.303802" rpy="0 0 0"/>
-    <geometry>
-      <mesh filename="package://marta_description/meshes/l_feet_1.stl" scale="0.001 0.001 0.001"/>
-    </geometry>
+    <xacro:if value="${'$(arg foot_collision)' == 'box'}">
+      <!-- Mesma caixa envolvente da sola do STL (bbox medido da malha). -->
+      <origin xyz="0.02445 0 -0.013" rpy="0 0 0"/>
+      <geometry>
+        <box size="0.1399 0.070 0.048"/>
+      </geometry>
+    </xacro:if>
+    <xacro:unless value="${'$(arg foot_collision)' == 'box'}">
+      <origin xyz="0.017701 -0.039506 0.303802" rpy="0 0 0"/>
+      <geometry>
+        <mesh filename="package://marta_description/meshes/l_feet_1.stl" scale="0.001 0.001 0.001"/>
+      </geometry>
+    </xacro:unless>
     <surface>
       <contact>
           <ode>
-            <!-- <max_vel>0</max_vel> -->
-            <kp>1e25</kp>
-            <kd>1e23</kd>
+            <!-- Mesma fonte que o bloco <gazebo reference="*_feet_1"> em
+                 marta.gazebo: antes havia 1e25/1e23 aqui e 1e6/1e4 la, valores
+                 conflitantes para a mesma superficie. -->
+            <kp>${contact_kp}</kp>
+            <kd>${contact_kd}</kd>
           </ode>
         </contact>
@@ -437,14 +505,25 @@
   </visual>
   <collision>
-    <origin xyz="0.017701 0.039494 0.303802" rpy="0 0 0"/>
-    <geometry>
-      <mesh filename="package://marta_description/meshes/r_feet_1.stl" scale="0.001 0.001 0.001"/>
-    </geometry>
+    <xacro:if value="${'$(arg foot_collision)' == 'box'}">
+      <!-- Mesma caixa envolvente da sola do STL (bbox medido da malha). -->
+      <origin xyz="0.02445 0 -0.013" rpy="0 0 0"/>
+      <geometry>
+        <box size="0.1399 0.070 0.048"/>
+      </geometry>
+    </xacro:if>
+    <xacro:unless value="${'$(arg foot_collision)' == 'box'}">
+      <origin xyz="0.017701 0.039494 0.303802" rpy="0 0 0"/>
+      <geometry>
+        <mesh filename="package://marta_description/meshes/r_feet_1.stl" scale="0.001 0.001 0.001"/>
+      </geometry>
+    </xacro:unless>
     <surface>
       <contact>
           <ode>
-            <!-- <max_vel>0</max_vel> -->
-            <kp>1e25</kp>
-            <kd>1e23</kd>
+            <!-- Mesma fonte que o bloco <gazebo reference="*_feet_1"> em
+                 marta.gazebo: antes havia 1e25/1e23 aqui e 1e6/1e4 la, valores
+                 conflitantes para a mesma superficie. -->
+            <kp>${contact_kp}</kp>
+            <kd>${contact_kd}</kd>
           </ode>
         </contact>

File: urdf/marta_joints.xacro (robot description, xacro)
@@ -9,6 +9,6 @@
   <child link="neck_1"/>
   <axis xyz="-0.0 0.0 -1.0"/>
-  <!-- <dynamics damping="0.1" /> -->
-  <limit lower="-3.14159" upper="3.14159" effort="1000.0" velocity="0.01"/>
+  <dynamics damping="${joint_damping}" friction="${joint_friction}"/>
+  <limit lower="-3.14159" upper="3.14159" effort="${joint_effort}" velocity="0.01"/>
 </joint>
 <joint name="head_tilt_link" type="revolute">
@@ -17,6 +17,6 @@
   <child link="head_1"/>
   <axis xyz="-0.0 -1.0 -0.0"/>
-  <!-- <dynamics damping="0.1" /> -->
-  <limit lower="-3.14159" upper="3.14159" effort="1000.0" velocity="0.01"/>
+  <dynamics damping="${joint_damping}" friction="${joint_friction}"/>
+  <limit lower="-3.14159" upper="3.14159" effort="${joint_effort}" velocity="0.01"/>
 </joint>
 <joint name="r_hip_yaw_link" type="revolute">
@@ -25,6 +25,6 @@
   <child link="r_hip_1"/>
   <axis xyz="-0.0 0.0 -1.0"/>
-  <!-- <dynamics damping="0.1" /> -->
-  <limit lower="-3.14159" upper="3.14159" effort="1000.0" velocity="0.01"/>
+  <dynamics damping="${joint_damping}" friction="${joint_friction}"/>
+  <limit lower="-3.14159" upper="3.14159" effort="${joint_effort}" velocity="0.01"/>
 </joint>
 <joint name="l_hip_yaw_link" type="revolute">
@@ -33,6 +33,6 @@
   <child link="l_hip_1"/>
   <axis xyz="0.0 0.0 -1.0"/>
-  <!-- <dynamics damping="0.1" /> -->
-  <limit lower="-3.14159" upper="3.14159" effort="1000.0" velocity="0.01"/>
+  <dynamics damping="${joint_damping}" friction="${joint_friction}"/>
+  <limit lower="-3.14159" upper="3.14159" effort="${joint_effort}" velocity="0.01"/>
 </joint>
 <joint name="l_hip_roll_link" type="revolute">
@@ -41,6 +41,6 @@
   <child link="l_waist_1"/>
   <axis xyz="1.0 -0.0 0.0"/>
-  <!-- <dynamics damping="0.1" /> -->
-  <limit lower="-3.14159" upper="3.14159" effort="1000.0" velocity="0.01"/>
+  <dynamics damping="${joint_damping}" friction="${joint_friction}"/>
+  <limit lower="-3.14159" upper="3.14159" effort="${joint_effort}" velocity="0.01"/>
 </joint>
 <joint name="r_hip_roll_link" type="revolute">
@@ -49,6 +49,6 @@
   <child link="r_waist_1"/>
   <axis xyz="1.0 0.0 -0.0"/>
-  <!-- <dynamics damping="0.1" /> -->
-  <limit lower="-3.14159" upper="3.14159" effort="1000.0" velocity="0.01"/>
+  <dynamics damping="${joint_damping}" friction="${joint_friction}"/>
+  <limit lower="-3.14159" upper="3.14159" effort="${joint_effort}" velocity="0.01"/>
 </joint>
 <joint name="r_hip_pitch_link" type="revolute">
@@ -57,6 +57,6 @@
   <child link="r_thigh_1"/>
   <axis xyz="0.0 1.0 -0.0"/>
-  <!-- <dynamics damping="0.1" /> -->
-  <limit lower="-3.14159" upper="3.14159" effort="1000.0" velocity="0.01"/>
+  <dynamics damping="${joint_damping}" friction="${joint_friction}"/>
+  <limit lower="-3.14159" upper="3.14159" effort="${joint_effort}" velocity="0.01"/>
 </joint>
 <joint name="l_hip_pitch_link" type="revolute">
@@ -65,6 +65,6 @@
   <child link="l_thigh_1"/>
   <axis xyz="0.0 1.0 0.0"/>
-  <!-- <dynamics damping="0.1" /> -->
-  <limit lower="-3.14159" upper="3.14159" effort="1000.0" velocity="0.01"/>
+  <dynamics damping="${joint_damping}" friction="${joint_friction}"/>
+  <limit lower="-3.14159" upper="3.14159" effort="${joint_effort}" velocity="0.01"/>
 </joint>
 <joint name="r_knee_link" type="revolute">
@@ -73,6 +73,6 @@
   <child link="r_shin_1"/>
   <axis xyz="-0.0 1.0 -0.0"/>
-  <!-- <dynamics damping="0.1" /> -->
-  <limit lower="-3.14159" upper="3.14159" effort="1000.0" velocity="0.01"/>
+  <dynamics damping="${joint_damping}" friction="${joint_friction}"/>
+  <limit lower="-3.14159" upper="3.14159" effort="${joint_effort}" velocity="0.01"/>
 </joint>
 <joint name="l_knee_link" type="revolute">
@@ -81,6 +81,6 @@
   <child link="l_shin_1"/>
   <axis xyz="0.0 1.0 0.0"/>
-  <!-- <dynamics damping="0.1" /> -->
-  <limit lower="-3.14159" upper="3.14159" effort="1000.0" velocity="0.01"/>
+  <dynamics damping="${joint_damping}" friction="${joint_friction}"/>
+  <limit lower="-3.14159" upper="3.14159" effort="${joint_effort}" velocity="0.01"/>
 </joint>
 <joint name="l_ank_pitch_link" type="revolute">
@@ -89,6 +89,6 @@
   <child link="l_ankle_1"/>
   <axis xyz="-0.0 1.0 -0.0"/>
-  <!-- <dynamics damping="0.1" /> -->
-  <limit lower="-3.14159" upper="3.14159" effort="1000.0" velocity="0.01"/>
+  <dynamics damping="${joint_damping}" friction="${joint_friction}"/>
+  <limit lower="-3.14159" upper="3.14159" effort="${joint_effort}" velocity="0.01"/>
 </joint>
 <joint name="r_ank_pitch_link" type="revolute">
@@ -97,6 +97,6 @@
   <child link="r_ankle_1"/>
   <axis xyz="-0.0 1.0 0.0"/>
-  <!-- <dynamics damping="0.1" /> -->
-  <limit lower="-3.14159" upper="3.14159" effort="1000.0" velocity="0.01"/>
+  <dynamics damping="${joint_damping}" friction="${joint_friction}"/>
+  <limit lower="-3.14159" upper="3.14159" effort="${joint_effort}" velocity="0.01"/>
 </joint>
 <joint name="r_ank_roll_link" type="revolute">
@@ -105,6 +105,6 @@
   <child link="r_feet_1"/>
   <axis xyz="1.0 0.0 -0.0"/>
-  <!-- <dynamics damping="0.1" /> -->
-  <limit lower="-3.14159" upper="3.14159" effort="1000.0" velocity="0.01"/>
+  <dynamics damping="${joint_damping}" friction="${joint_friction}"/>
+  <limit lower="-3.14159" upper="3.14159" effort="${joint_effort}" velocity="0.01"/>
 </joint>
 <joint name="l_sho_pitch_link" type="revolute">
@@ -113,6 +113,6 @@
   <child link="l_shoulder_1"/>
   <axis xyz="0.0 1.0 0.0"/>
-  <!-- <dynamics damping="0.1" /> -->
-  <limit lower="-3.14159" upper="3.14159" effort="1000.0" velocity="0.01"/>
+  <dynamics damping="${joint_damping}" friction="${joint_friction}"/>
+  <limit lower="-3.14159" upper="3.14159" effort="${joint_effort}" velocity="0.01"/>
 </joint>
 <joint name="r_sho_pitch_link" type="revolute">
@@ -121,6 +121,6 @@
   <child link="r_shoulder_1"/>
   <axis xyz="-0.0 1.0 -0.0"/>
-  <!-- <dynamics damping="0.1" /> -->
-  <limit lower="-3.14159" upper="3.14159" effort="1000.0" velocity="0.01"/>
+  <dynamics damping="${joint_damping}" friction="${joint_friction}"/>
+  <limit lower="-3.14159" upper="3.14159" effort="${joint_effort}" velocity="0.01"/>
 </joint>
 <joint name="l_sho_roll_link" type="revolute">
@@ -129,6 +129,6 @@
   <child link="l_arm_1"/>
   <axis xyz="-1.0 -0.0 -0.0"/>
-  <!-- <dynamics damping="0.1" /> -->
-  <limit lower="-3.14159" upper="3.14159" effort="1000.0" velocity="0.01"/>
+  <dynamics damping="${joint_damping}" friction="${joint_friction}"/>
+  <limit lower="-3.14159" upper="3.14159" effort="${joint_effort}" velocity="0.01"/>
 </joint>
 <joint name="r_sho_roll_link" type="revolute">
@@ -137,6 +137,6 @@
   <child link="r_arm_1"/>
   <axis xyz="-1.0 0.0 -0.0"/>
-  <!-- <dynamics damping="0.1" /> -->
-  <limit lower="-3.14159" upper="3.14159" effort="1000.0" velocity="0.01"/>
+  <dynamics damping="${joint_damping}" friction="${joint_friction}"/>
+  <limit lower="-3.14159" upper="3.14159" effort="${joint_effort}" velocity="0.01"/>
 </joint>
 <joint name="l_ank_roll_link" type="revolute">
@@ -145,6 +145,6 @@
   <child link="l_feet_1"/>
   <axis xyz="1.0 -0.0 0.0"/>
-  <!-- <dynamics damping="0.1" /> -->
-  <limit lower="-3.14159" upper="3.14159" effort="1000.0" velocity="0.01"/>
+  <dynamics damping="${joint_damping}" friction="${joint_friction}"/>
+  <limit lower="-3.14159" upper="3.14159" effort="${joint_effort}" velocity="0.01"/>
 </joint>
 <joint name="r_el_link" type="revolute">
@@ -153,6 +153,6 @@
   <child link="r_hand_1"/>
   <axis xyz="0.0 1.0 -0.0"/>
-  <!-- <dynamics damping="0.1" /> -->
-  <limit lower="-3.14159" upper="3.14159" effort="1000.0" velocity="0.01"/>
+  <dynamics damping="${joint_damping}" friction="${joint_friction}"/>
+  <limit lower="-3.14159" upper="3.14159" effort="${joint_effort}" velocity="0.01"/>
 </joint>
 <joint name="l_el_link" type="revolute">
@@ -161,6 +161,6 @@
   <child link="l_hand_1"/>
   <axis xyz="-0.0 1.0 0.0"/>
-  <!-- <dynamics damping="0.1" /> -->
-  <limit lower="-3.14159" upper="3.14159" effort="1000.0" velocity="0.01"/>
+  <dynamics damping="${joint_damping}" friction="${joint_friction}"/>
+  <limit lower="-3.14159" upper="3.14159" effort="${joint_effort}" velocity="0.01"/>
 </joint>
 </robot>
